Commit message: fix typo cylinder radius

File: Project 4 - Where Am I/my_robot/urdf/my_robot.xacro (robot description, xacro)
@@ -22,5 +22,5 @@
       <origin xyz="0 0 0" rpy=" 0 0 0"/>
       <geometry>
-        <cylinder raduis="0.21" length="0.1"/>
+        <cylinder radius="0.21" length="0.1"/>
       </geometry>
     </collision>
@@ -28,5 +28,5 @@
       <origin xyz="0 0 0" rpy=" 0 0 0"/>
       <geometry>
-        <cylinder raduis="0.21" length="0.1"/>
+        <cylinder radius="0.21" length="0.1"/>
       </geometry>
     </visual>

Commit message: Update map information

File: Project 4 - Where Am I/my_robot/urdf/my_robot.xacro (robot description, xacro)
@@ -4,5 +4,5 @@
   <link name="robot_footprint"></link>
   <joint name="robot_footprint_joint" type="fixed">
-    <origin xyz="0 0 0" rpy="0 0 0" />
+    <origin xyz="-4 -6 0" rpy="0 0 0" />
     <parent link="robot_footprint"/>
     <child link="chassis" />

Commit message: Adjust robot position

File: Project 4 - Where Am I/my_robot/urdf/my_robot.xacro (robot description, xacro)
@@ -4,5 +4,5 @@
   <link name="robot_footprint"></link>
   <joint name="robot_footprint_joint" type="fixed">
-    <origin xyz="-4 -6 0" rpy="0 0 0" />
+    <origin xyz="0 0 0" rpy="0 0 0" />
     <parent link="robot_footprint"/>
     <child link="chassis" />
